File: kicad/board/board.kicad_pcb (KiCad board)
At the start: 2 copper layers, 126.9 x 103.7 mm, 44 parts

Commit message: Finished PCB traces
Parts:
- moved D1 205.3 mm to (137.4, 162.7)
- moved D10 205.3 mm to (192.4, 158.5)
- moved D11 205.3 mm to (194.0, 140.6)
- moved D12 205.3 mm to (195.6, 122.6)
- moved D13 205.3 mm to (210.2, 162.1)
- moved D14 205.3 mm to (211.8, 144.1)
- moved D15 205.3 mm to (213.3, 126.2)
- moved D16 205.3 mm to (201.6, 180.4)
- moved D17 205.3 mm to (219.9, 186.2)
- moved D18 205.3 mm to (236.2, 196.3)
- moved D2 205.3 mm to (137.4, 144.7)
- moved D3 205.3 mm to (137.4, 126.7)
- moved D4 205.3 mm to (156.7, 154.4)
- moved D5 205.3 mm to (158.2, 136.4)
- moved D6 205.3 mm to (159.8, 118.5)
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Routing:
- net R2: track 0.00 -> 135.8 mm, vias 0 -> 4
- net R3: track 0.00 -> 126.4 mm
- net C0: track 95.4 -> 193.8 mm
- net R1: track 26.3 -> 118.3 mm, vias 2 -> 5
- net C1: track 100.4 -> 173.9 mm, vias 1 -> 2
- net C2: track 198.7 -> 247.8 mm
- net C3: track 183.9 -> 213.6 mm, vias 1 -> 2
- net C4: track 186.9 -> 199.8 mm, vias 1 -> 2
- net Net-(JST2-Pin_1): vias 2 -> 0
